File: audio_circuit/Peachy1-99-6-f.sch (EAGLE design)
At the start: 131 parts, among them CON1 CUI-SJ-3523-SMT, CON2 CUI-SJ-3523-SMT, IC1 LM324ADR, IC2 LM324ADR, IC3 LM324ADR, IC4 LMC7101, IC5 LMC7101, Q1 DMG4406LSS, Q2 DMG4406LSS, Q3 BC857CT, Q4 MMBT3904, U1 ADP1613, U2 ADP2300, X10 TSW-102-02-S-S, X2 JUMPER-31-2, X3 JUMPER-31-2, X6 OSTTE030104, X7 TSW-103-02-S-S, X9 TSW-103-02-S-S

Commit message: Updated Scotts audio board files with his latest
Parts:
- C4, C6: value .01uF -> 0.01uF
- CBST-NEG: value 0.1uF 6.3v -> 0.1uF
- CC-NEG: value 1uF 16V low ESR -> 1uF
- CIN-NEG: value 4.7uF Low ESR -> 4.7uF
- D1-NEG: value MBR0520LT1G -> MBR0520
- R11: value 1k37 -> 1k37 1%
- R12: value 2k55 -> 2k55 1%
- R16: MPN RC0805JR-07220RL -> RMCF0805JT220R
- R19, R20, R24, R25: value 6k8 -> 6k8 1%
- R30, REN: value 10K -> 10k
Changed lines of the file:
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@@
 <part name="GND11" library="Scott" deviceset="GND" device=""/>
 <part name="GND12" library="Scott" deviceset="GND" device=""/>
-<part name="R25" library="Scott" deviceset="R-US_" device="R0805" value="6k8">
-<attribute name="MPN" value="RC0805FR-076K8L"/>
-</part>
-<part name="R24" library="Scott" deviceset="R-US_" device="R0805" value="6k8">
-<attribute name="MPN" value="RC0805FR-076K8L"/>
-</part>
-<part name="R20" library="Scott" deviceset="R-US_" device="R0805" value="6k8">
-<attribute name="MPN" value="RC0805FR-076K8L"/>
-</part>
-<part name="R19" library="Scott" deviceset="R-US_" device="R0805" value="6k8">
+<part name="R25" library="Scott" deviceset="R-US_" device="R0805" value="6k8 1%">
+<attribute name="MPN" value="RC0805FR-076K8L"/>
+</part>
+<part name="R24" library="Scott" deviceset="R-US_" device="R0805" value="6k8 1%">
+<attribute name="MPN" value="RC0805FR-076K8L"/>
+</part>
+<part name="R20" library="Scott" deviceset="R-US_" device="R0805" value="6k8 1%">
+<attribute name="MPN" value="RC0805FR-076K8L"/>
+</part>
+<part name="R19" library="Scott" deviceset="R-US_" device="R0805" value="6k8 1%">
 <attribute name="MPN" value="RC0805FR-076K8L"/>
 </part>
@@
 <attribute name="MPN" value="RC0805FR-071K37L"/>
 </part>
-<part name="C6" library="Scott" deviceset="C-US" device="0805" value=".01uF">
+<part name="C6" library="Scott" deviceset="C-US" device="0805" value="0.01uF">
 <attribute name="MPN" value="CL21B103KBANNNC"/>
 </part>
-<part name="C4" library="Scott" deviceset="C-US" device="0805" value=".01uF">
+<part name="C4" library="Scott" deviceset="C-US" device="0805" value="0.01uF">
 <attribute name="MPN" value="CL21B103KBANNNC"/>
 </part>
@@
 <part name="GND20" library="Scott" deviceset="GND" device=""/>
 <part name="GND25" library="Scott" deviceset="GND" device=""/>
-<part name="R30" library="Scott" deviceset="R-US_" device="R0805" value="10K">
+<part name="R30" library="Scott" deviceset="R-US_" device="R0805" value="10k">
 <attribute name="MPN" value="RMCF0805JT10K0"/>
 </part>
@@
 <attribute name="MPN" value="DMG4406LSS-13"/>
 </part>
-<part name="R11" library="Scott" deviceset="R-US_" device="R0805" value="1k37">
+<part name="R11" library="Scott" deviceset="R-US_" device="R0805" value="1k37 1%">
 <attribute name="MPN" value="RC0805FR-071K37L"/>
 </part>
-<part name="R12" library="Scott" deviceset="R-US_" device="R0805" value="2k55">
+<part name="R12" library="Scott" deviceset="R-US_" device="R0805" value="2k55 1%">
 <attribute name="MPN" value="RC0805FR-072K55L"/>
 </part>
@@
 <attribute name="MPN" value="RMCF0805JT1R00 "/>
 </part>
-<part name="REN" library="Scott" deviceset="R-US_" device="R0805" value="10K">
+<part name="REN" library="Scott" deviceset="R-US_" device="R0805" value="10k">
 <attribute name="MPN" value="RMCF0805JT10K0"/>
 </part>
@@
 <attribute name="MPN" value="ADP2300AUJZ-R7"/>
 </part>
-<part name="CIN-NEG" library="Scott" deviceset="C-US" device="0805" value="4.7uF Low ESR">
+<part name="CIN-NEG" library="Scott" deviceset="C-US" device="0805" value="4.7uF">
 <attribute name="MPN" value="CL21A475KOFNNNE"/>
 </part>
-<part name="CC-NEG" library="Scott" deviceset="C-US" device="0805" value="1uF 16V low ESR">
+<part name="CC-NEG" library="Scott" deviceset="C-US" device="0805" value="1uF">
 <attribute name="MPN" value="CL21B105KBFNNNE"/>
 </part>
@@
 <attribute name="MPN" value="CL21B106KQQNNNE"/>
 </part>
-<part name="CBST-NEG" library="Scott" deviceset="C-US" device="0805" value="0.1uF 6.3v">
+<part name="CBST-NEG" library="Scott" deviceset="C-US" device="0805" value="0.1uF">
 <attribute name="MPN" value="CL21B104KACNNNC"/>
 </part>
@@
 <attribute name="MPN" value="LQH32PN6R8NN0"/>
 </part>
-<part name="D1-NEG" library="Scott" deviceset="SCHOTTKY" device="SOD123" value="MBR0520LT1G">
+<part name="D1-NEG" library="Scott" deviceset="SCHOTTKY" device="SOD123" value="MBR0520">
 <attribute name="MPN" value="MBR0520LT3G"/>
 </part>
@@
 </part>
 <part name="R16" library="Scott" deviceset="R-US_" device="R0805" value="220R">
-<attribute name="MPN" value="RC0805JR-07220RL"/>
+<attribute name="MPN" value="RMCF0805JT220R"/>
 </part>
 <part name="R17" library="Scott" deviceset="R-US_" device="R0805" value="1k2">
